File: tubeScreamer.kicad_pcb (KiCad board)
At the start: 2 copper layers, 100 x 100 mm, 51 parts, among them J1 IN, J2 IN, J3 OUT, J4 9V IN, J5 OUT, Q1 MMBT2222A, Q2 MMBT2222A, U1 TL072, U2 TL072

Commit message: test commit
Parts:
- Distortion1: footprint digikey-footprints:Potentiometer_P120PK-Y25BR10K -> Rotary_Encoder:RotaryEncoder_Bourns_Vertical_PEC12R-3x17F-Nxxxx
- moved Distortion1 1.40 mm to (125.5, 71.7), turned to 90 degrees
