File: tubeScreamer.kicad_sch (KiCad schematic)
At the start: 51 parts, among them J1 IN, J2 IN, J3 OUT, J4 9V IN, J5 OUT, Q1 MMBT2222A, Q2 MMBT2222A, U1 TL072, U2 TL072

Commit message: test commit
Parts:
- Distortion1: footprint digikey-footprints:Potentiometer_P120PK-Y25BR10K -> Rotary_Encoder:RotaryEncoder_Bourns_Vertical_PEC12R-3x17F-Nxxxx
Changed lines of the file:
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@@
 	)
 	(junction
+		(at 121.92 121.92)
+		(diameter 0)
+		(color 0 0 0 0)
+	)
+	(junction
 		(at 106.68 121.92)
 		(diameter 0)
@@
 	)
 	(junction
-		(at 121.92 121.92)
-		(diameter 0)
-		(color 0 0 0 0)
-	)
-	(junction
 		(at 62.23 85.09)
 		(diameter 0)
@@
 	(wire
 		(pts
-			(xy 121.92 121.92) (xy 121.92 129.54)
+			(xy 33.02 40.64) (xy 33.02 44.45)
 		)
 		(stroke
@@
 	(wire
 		(pts
-			(xy 33.02 40.64) (xy 33.02 44.45)
+			(xy 227.33 101.6) (xy 231.14 101.6)
 		)
 		(stroke
@@
 	(wire
 		(pts
-			(xy 227.33 101.6) (xy 231.14 101.6)
+			(xy 114.3 97.79) (xy 114.3 96.52)
 		)
 		(stroke
@@
 	(wire
 		(pts
-			(xy 114.3 97.79) (xy 114.3 96.52)
+			(xy 227.33 85.09) (xy 227.33 87.63)
 		)
 		(stroke
@@
 	(wire
 		(pts
-			(xy 227.33 85.09) (xy 227.33 87.63)
+			(xy 30.48 29.21) (xy 30.48 34.29)
 		)
 		(stroke
@@
 	(wire
 		(pts
-			(xy 30.48 29.21) (xy 30.48 34.29)
+			(xy 205.74 93.98) (xy 201.93 93.98)
 		)
 		(stroke
@@
 	(wire
 		(pts
-			(xy 205.74 93.98) (xy 201.93 93.98)
+			(xy 36.83 80.01) (xy 36.83 87.63)
 		)
 		(stroke
@@
 	(wire
 		(pts
-			(xy 36.83 80.01) (xy 36.83 87.63)
+			(xy 114.3 133.35) (xy 118.11 133.35)
 		)
 		(stroke
@@
 	(wire
 		(pts
-			(xy 118.11 133.35) (xy 114.3 133.35)
-		)
-		(stroke
-			(width 0)
-			(type default)
-		)
-	)
-	(wire
-		(pts
 			(xy 121.92 101.6) (xy 121.92 91.44)
 		)
@@
 	(wire
 		(pts
+			(xy 121.92 121.92) (xy 121.92 129.54)
+		)
+		(stroke
+			(width 0)
+			(type default)
+		)
+	)
+	(wire
+		(pts
 			(xy 50.8 124.46) (xy 50.8 137.16)
 		)
@@
 			)
 		)
-		(property "Footprint" "digikey-footprints:Potentiometer_P120PK-Y25BR10K"
+		(property "Footprint" "Rotary_Encoder:RotaryEncoder_Bourns_Vertical_PEC12R-3x17F-Nxxxx"
 			(at 121.92 133.35 0)
 			(effects
